File: pcb_files/Remote/IRstart - Remote.kicad_pcb (KiCad board)
At the start: 2 copper layers, 40 x 59.4 mm, 35 parts, among them SW1 SW_DIP_x02, SW2 SW_DIP_x02, SW3 SW_DPDT_x2

Commit message: Avanza con el diseño de la PCB
Parts:
- removed JP2: Jumper_2_Bridged, Jumper:SolderJumper-2_P1.3mm_Bridged_Pad1.0x1.5mm
- added C4: 10uF, Capacitor_SMD:C_0805_2012Metric_Pad1.18x1.45mm_HandSolder, F.Cu at (166.6, 116.6)
- added C5: 10uF, Capacitor_SMD:C_0805_2012Metric_Pad1.18x1.45mm_HandSolder, F.Cu at (170.7, 116.6)
- added D1: LED, LED_SMD:LED_0805_2012Metric_Pad1.15x1.40mm_HandSolder, F.Cu at (135.6, 120.8)
- added D2: LED, LED_SMD:LED_0805_2012Metric_Pad1.15x1.40mm_HandSolder, F.Cu at (135.6, 122.9)
- added LDO1: ~, Package_TO_SOT_SMD:SOT-23-5_HandSoldering, F.Cu at (140.7, 122.3)
- added R18: 1K5, Resistor_SMD:R_0805_2012Metric_Pad1.20x1.40mm_HandSolder, F.Cu at (168.7, 116.6)
- added R19: 0, Resistor_SMD:R_0805_2012Metric_Pad1.20x1.40mm_HandSolder, F.Cu at (153.5, 94.6)
- added R4: 1K, Resistor_SMD:R_0805_2012Metric_Pad1.20x1.40mm_HandSolder, F.Cu at (141.4, 111.3)
- added R5: 1K, Resistor_SMD:R_0805_2012Metric_Pad1.20x1.40mm_HandSolder, F.Cu at (141.4, 115.8)
- added TP4056: ~, Package_SO:SOP-8_3.9x4.9mm_P1.27mm, F.Cu at (168.7, 110.4)
- added kibuzzard-6637BADB: G***, kibuzzard-6637BADB, F.Cu at (140.8, 82.0)
- added kibuzzard-6637BAEA: G***, kibuzzard-6637BAEA, F.Cu at (153.5, 80.5)
- added kibuzzard-6637BBE8: G***, kibuzzard-6637BBE8, F.Cu at (136.3, 107.4)
- added kibuzzard-6637BC1A: G***, kibuzzard-6637BC1A, F.Cu at (136.3, 118.1)
- added kibuzzard-6637BD08: G***, kibuzzard-6637BD08, F.Cu at (166.8, 82.2)
- added kibuzzard-6637DAEE: G***, kibuzzard-6637DAEE, B.Cu at (159.8, 122.2)
- BT1: footprint Battery:BatteryHolder_Keystone_3002_1x2032 -> custom_footprints:Leds_IR_Remote
- LED1, LED2, LED3: footprint LED_SMD:LED_PLCC-2_3x2mm_KA -> custom_footprints:Leds_IR_Remote
- NEO1, NEO2, NEO3: footprint LED_SMD:LED_WS2812B-2020_PLCC4_2.0x2.0mm -> custom_footprints:LED_WS2812B_2.0x2.0mm
- moved BT1 28.1 mm to (159.8, 126.7)
- moved R6 15.9 mm to (144.5, 102.3)
- moved R7 15.8 mm to (146.8, 102.3)
- moved R17 15.4 mm to (162.5, 102.3)
- moved R16 15.3 mm to (160.3, 102.3)
- moved R8 13.9 mm to (151.2, 102.3)
- moved ESP1 13.1 mm to (153.5, 124.7)
- moved R15 11.7 mm to (153.5, 102.3)
- moved R11 9.41 mm to (158.1, 102.3), turned to -90 degrees
- moved R10 9.33 mm to (155.8, 102.3), turned to -90 degrees
- moved MOSFET1 9.26 mm to (150.0, 93.7)
- moved MOSFET2 9.26 mm to (157.1, 93.7)
- moved R1 8.17 mm to (144.5, 98.3), turned to -90 degrees
- moved R2 8.13 mm to (146.8, 98.2), turned to -90 degrees
- moved R3 8.06 mm to (149.0, 98.2), turned to -90 degrees
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Connections:
- BT1 pad 1: Net-(BT1-+) -> /BATT
- ESP1 pad 9: unconnected-(ESP1-5V-Pad9) -> +5V
- R15 pad 1: Net-(LED3-GND) -> Net-(LED2-GND)
- R2 pad 1: Net-(LED2-GND) -> Net-(LED3-GND)
- R3 pad 1: Net-(LED3-GND) -> Net-(LED2-GND)
- SW3 pad 1: unconnected-(SW3A-A-Pad1) -> /BATT
- SW3 pad 2: +3.3V -> Net-(LDO1-CE)
- SW3 pad 3: Net-(BT1-+) -> unconnected-(SW3A-C-Pad3)
Routing:
- net +3.3V: track 0.00 -> 202.3 mm, vias 0 -> 6
- net GND: track 0.00 -> 181.3 mm, vias 0 -> 24
- net +5V: track 0.00 -> 68.4 mm, vias 0 -> 7
- net /BATT: track 0.00 -> 63.3 mm, vias 0 -> 2
- net /READY_BTN: track 0.00 -> 62.1 mm, vias 0 -> 5
- net /STOP_BTN: track 0.00 -> 57.6 mm, vias 0 -> 5
- net /START_BTN: track 0.00 -> 49.6 mm, vias 0 -> 4
- net Net-(LED2-GND): track 0.00 -> 44.8 mm, vias 0 -> 2
- net /RGBs: track 0.00 -> 43.6 mm, vias 0 -> 2
- net /LED_CARGA: track 0.00 -> 39.8 mm, vias 0 -> 2
- net /LED_CARGADO: track 0.00 -> 39.7 mm, vias 0 -> 2
- net /SWITCH4: track 0.00 -> 30.5 mm
- net Net-(D1-A): track 0.00 -> 27.4 mm
- net /SWITCH3: track 0.00 -> 26.0 mm
- net Net-(LED3-GND): track 0.00 -> 23.6 mm, vias 0 -> 2
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- added copper zone on B.Cu, net GND
- added copper zone on F.Cu, net GND
Other:
- outline, holes or cut-outs redrawn
- board text added: "ESP32"
